Commit message: pose finished

File: assets/franka/urdf/franka_panda_phase4.urdf (robot description, URDF)
Before this commit: robot phase4_franka_panda, 12 links, 11 joints
Links:
- link panda_hand: geometry collision mesh filename=/home/ziyaochen/torc_franka_lift3d_pipeline_v2/assets/frank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; visual mesh filename=/home/ziyaochen/torc_franka_lift3d_pipeline_v2/assets/frank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
- link panda_leftfinger: geometry collision mesh filename=/home/ziyaochen/torc_franka_lift3d_pipeline_v2/assets/frank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; visual mesh filename=/home/ziyaochen/torc_franka_lift3d_pipeline_v2/assets/frank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
- link panda_link0: geometry collision mesh filename=/home/ziyaochen/torc_franka_lift3d_pipeline_v2/assets/frank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; visual mesh filename=/home/ziyaochen/torc_franka_lift3d_pipeline_v2/assets/frank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
- link panda_link1: geometry collision mesh filename=/home/ziyaochen/torc_franka_lift3d_pipeline_v2/assets/frank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; visual mesh filename=/home/ziyaochen/torc_franka_lift3d_pipeline_v2/assets/frank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
- link panda_link2: geometry collision mesh filename=/home/ziyaochen/torc_franka_lift3d_pipeline_v2/assets/frank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; visual mesh filename=/home/ziyaochen/torc_franka_lift3d_pipeline_v2/assets/frank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
- link panda_link3: geometry collision mesh filename=/home/ziyaochen/torc_franka_lift3d_pipeline_v2/assets/frank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; visual mesh filename=/home/ziyaochen/torc_franka_lift3d_pipeline_v2/assets/frank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
- link panda_link4: geometry collision mesh filename=/home/ziyaochen/torc_franka_lift3d_pipeline_v2/assets/frank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; visual mesh filename=/home/ziyaochen/torc_franka_lift3d_pipeline_v2/assets/frank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
- link panda_link5: geometry collision mesh filename=/home/ziyaochen/torc_franka_lift3d_pipeline_v2/assets/frank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; visual mesh filename=/home/ziyaochen/torc_franka_lift3d_pipeline_v2/assets/frank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
- link panda_link6: geometry collision mesh filename=/home/ziyaochen/torc_franka_lift3d_pipeline_v2/assets/frank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; visual mesh filename=/home/ziyaochen/torc_franka_lift3d_pipeline_v2/assets/frank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
- link panda_link7: geometry collision mesh filename=/home/ziyaochen/torc_franka_lift3d_pipeline_v2/assets/frank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; visual mesh filename=/home/ziyaochen/torc_franka_lift3d_pipeline_v2/assets/frank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
- link panda_rightfinger: geometry collision mesh filename=/home/ziyaochen/torc_franka_lift3d_pipeline_v2/assets/frank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; visual mesh filename=/home/ziyaochen/torc_franka_lift3d_pipeline_v2/assets/frank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
